File: project.sch (KiCad schematic (older format))
At the start: 30 parts, among them J1 Conn_01x02, J2 Conn_01x15, J3 Conn_01x15, J4 Conn_01x02, J5 Conn_01x02, J6 Conn_01x02, U1 DRV8870DDA, U2 DRV8870DDA, U3 DRV8870DDA

Commit message: Add bom
Parts:
- A1: Digikey (none) -> https://www.digikey.ca/product-detail/en/sullins-connector-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; Notes (none) -> Digikey link is for female headers to connect to arduino, g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
- C1, C3, C5: Digikey (none) -> https://www.digikey.com/product-detail/en/kemet/C0603C104M5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
- C2, C4, C6: Digikey (none) -> https://www.digikey.com/product-detail/en/nichicon/UWT1H470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
- J1, J4, J5, J6: Mouser (none) -> https://www.mouser.ca/ProductDetail/Altech/30602?qs=sGAEpiM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
- J2, J3: Digikey (none) -> https://www.digikey.ca/product-detail/en/adam-tech/PH1-15-U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
- R1, R2, R3, R4, R5, R6: Digikey (none) -> https://www.digikey.com/product-detail/en/stackpole-electro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
- RV1: Digikey (none) -> https://www.digikey.ca/product-detail/en/bourns-inc/3266W-1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
- U1, U2, U3: Digikey (none) -> https://www.digikey.com/product-detail/en/texas-instruments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
Changed lines of the file:
@@
 F 3 "~" H 7700 4200 50  0001 C CNN
 F 4 "POWER IN" H 7780 4055 50  0000 L CNN "Purpose"
+F 5 "https://www.mouser.ca/ProductDetail/Altech/30602?qs=sGAEpiMZZMvlX3nhDDO4AL25%252B41q1QHAiP%252BMig2GC%2FM%3D" H 7700 4200 50  0001 C CNN "Mouser"
 	1    7700 4200
 	1    0    0    -1
@@
 F 3 "~" H 7700 3000 50  0001 C CNN
 F 4 "COIL X OUT" H 7780 2855 50  0000 L CNN "Purpose"
+F 5 "https://www.mouser.ca/ProductDetail/Altech/30602?qs=sGAEpiMZZMvlX3nhDDO4AL25%252B41q1QHAiP%252BMig2GC%2FM%3D" H 7700 3000 50  0001 C CNN "Mouser"
 	1    7700 3000
 	1    0    0    -1
@@
 F 2 "Potentiometer_THT:Potentiometer_Bourns_3266W_Vertical" H 6850 1850 50  0001 C CNN
 F 3 "~" H 6850 1850 50  0001 C CNN
+F 4 "https://www.digikey.ca/product-detail/en/bourns-inc/3266W-1-103LF/3266W-103LF-ND/1087907" H 6850 1850 50  0001 C CNN "Digikey"
 	1    6850 1850
 	1    0    0    -1
@@
 F 3 "~" H 2050 2350 50  0001 C CNN
 F 4 "CSR1206FKR300" H 2120 2259 50  0000 L CNN "Part Number"
+F 5 "https://www.digikey.com/product-detail/en/stackpole-electronics-inc/CSR1206FKR300/CSR1206FKR300CT-ND/1788117" H 2050 2350 50  0001 C CNN "Digikey"
 	1    2050 2350
 	1    0    0    -1
@@
 F 2 "Resistor_SMD:R_1206_3216Metric" V 1680 2350 50  0001 C CNN
 F 3 "~" H 1750 2350 50  0001 C CNN
+F 4 "https://www.digikey.com/product-detail/en/stackpole-electronics-inc/CSR1206FKR300/CSR1206FKR300CT-ND/1788117" H 1750 2350 50  0001 C CNN "Digikey"
 	1    1750 2350
 	1    0    0    -1
@@
 F 2 "Package_SO:Texas_HTSOP-8-1EP_3.9x4.9mm_P1.27mm_EP2.95x4.9mm_Mask2.4x3.1mm_ThermalVias" H 1600 1700 50  0001 C CNN
 F 3 "http://www.ti.com/lit/ds/symlink/drv8870.pdf" H 1250 2150 50  0001 C CNN
+F 4 "https://www.digikey.com/product-detail/en/texas-instruments/DRV8870DDAR/296-42660-1-ND/5455925" H 1500 1800 50  0001 C CNN "Digikey"
 	1    1500 1800
 	1    0    0    -1
@@
 F 3 "~" H 7700 3300 50  0001 C CNN
 F 4 "COIL Y OUT" H 7780 3155 50  0000 L CNN "Purpose"
+F 5 "https://www.mouser.ca/ProductDetail/Altech/30602?qs=sGAEpiMZZMvlX3nhDDO4AL25%252B41q1QHAiP%252BMig2GC%2FM%3D" H 7700 3300 50  0001 C CNN "Mouser"
 	1    7700 3300
 	1    0    0    -1
@@
 F 3 "~" H 7700 3600 50  0001 C CNN
 F 4 "COIL Z OUT" H 7780 3455 50  0000 L CNN "Purpose"
+F 5 "https://www.mouser.ca/ProductDetail/Altech/30602?qs=sGAEpiMZZMvlX3nhDDO4AL25%252B41q1QHAiP%252BMig2GC%2FM%3D" H 7700 3600 50  0001 C CNN "Mouser"
 	1    7700 3600
 	1    0    0    -1
@@
 F 3 "~" H 3950 2350 50  0001 C CNN
 F 4 "CSR1206FKR300" H 4020 2259 50  0000 L CNN "Part Number"
+F 5 "https://www.digikey.com/product-detail/en/stackpole-electronics-inc/CSR1206FKR300/CSR1206FKR300CT-ND/1788117" H 3950 2350 50  0001 C CNN "Digikey"
 	1    3950 2350
 	1    0    0    -1
@@
 F 2 "Resistor_SMD:R_1206_3216Metric" V 3580 2350 50  0001 C CNN
 F 3 "~" H 3650 2350 50  0001 C CNN
+F 4 "https://www.digikey.com/product-detail/en/stackpole-electronics-inc/CSR1206FKR300/CSR1206FKR300CT-ND/1788117" H 3650 2350 50  0001 C CNN "Digikey"
 	1    3650 2350
 	1    0    0    -1
@@
 F 2 "Package_SO:Texas_HTSOP-8-1EP_3.9x4.9mm_P1.27mm_EP2.95x4.9mm_Mask2.4x3.1mm_ThermalVias" H 3500 1700 50  0001 C CNN
 F 3 "http://www.ti.com/lit/ds/symlink/drv8870.pdf" H 3150 2150 50  0001 C CNN
+F 4 "https://www.digikey.com/product-detail/en/texas-instruments/DRV8870DDAR/296-42660-1-ND/5455925" H 3400 1800 50  0001 C CNN "Digikey"
 	1    3400 1800
 	1    0    0    -1
@@
 F 3 "~" H 5750 2350 50  0001 C CNN
 F 4 "CSR1206FKR300" H 5820 2259 50  0000 L CNN "Part Number"
+F 5 "https://www.digikey.com/product-detail/en/stackpole-electronics-inc/CSR1206FKR300/CSR1206FKR300CT-ND/1788117" H 5750 2350 50  0001 C CNN "Digikey"
 	1    5750 2350
 	1    0    0    -1
@@
 F 2 "Resistor_SMD:R_1206_3216Metric" V 5380 2350 50  0001 C CNN
 F 3 "~" H 5450 2350 50  0001 C CNN
+F 4 "https://www.digikey.com/product-detail/en/stackpole-electronics-inc/CSR1206FKR300/CSR1206FKR300CT-ND/1788117" H 5450 2350 50  0001 C CNN "Digikey"
 	1    5450 2350
 	1    0    0    -1
@@
 F 2 "Package_SO:Texas_HTSOP-8-1EP_3.9x4.9mm_P1.27mm_EP2.95x4.9mm_Mask2.4x3.1mm_ThermalVias" H 5300 1700 50  0001 C CNN
 F 3 "http://www.ti.com/lit/ds/symlink/drv8870.pdf" H 4950 2150 50  0001 C CNN
+F 4 "https://www.digikey.com/product-detail/en/texas-instruments/DRV8870DDAR/296-42660-1-ND/5455925" H 5200 1800 50  0001 C CNN "Digikey"
 	1    5200 1800
 	1    0    0    -1
@@
 F 2 "Module:Arduino_Nano" H 2200 5200 50  0001 C CIN
 F 3 "http://www.mouser.com/pdfdocs/Gravitech_Arduino_Nano3_0.pdf" H 2200 5200 50  0001 C CNN
+F 4 "https://www.digikey.ca/product-detail/en/sullins-connector-solutions/PPTC151LFBN-RC/S7013-ND/810153" H 2200 5200 50  0001 C CNN "Digikey"
+F 5 "Digikey link is for female headers to connect to arduino, get 2 if we don't have any lying around" H 2200 5200 50  0001 C CNN "Notes"
 	1    2200 5200
 	1    0    0    -1
@@
 F 3 "~" H 1850 1200 50  0001 C CNN
 F 4 "C0603C104M5RACTU" H 1850 1200 50  0001 C CNN "Part Number"
+F 5 "https://www.digikey.com/product-detail/en/kemet/C0603C104M5RACTU/399-7845-1-ND/3471568" H 1850 1200 50  0001 C CNN "Digikey"
 	1    1850 1200
 	1    0    0    -1
@@
 F 3 "" H 3750 1200 50  0001 C CNN
 F 4 "C0603C104M5RACTU" H 3750 1200 50  0001 C CNN "Part Number"
+F 5 "https://www.digikey.com/product-detail/en/kemet/C0603C104M5RACTU/399-7845-1-ND/3471568" H 3750 1200 50  0001 C CNN "Digikey"
 	1    3750 1200
 	1    0    0    -1
@@
 F 3 "~" H 5550 1200 50  0001 C CNN
 F 4 "C0603C104M5RACTU" H 5550 1200 50  0001 C CNN "Part Number"
+F 5 "https://www.digikey.com/product-detail/en/kemet/C0603C104M5RACTU/399-7845-1-ND/3471568" H 5550 1200 50  0001 C CNN "Digikey"
 	1    5550 1200
 	1    0    0    -1
@@
 F 2 "Connector_PinHeader_2.54mm:PinHeader_1x15_P2.54mm_Vertical" H 3850 5200 50  0001 C CNN
 F 3 "~" H 3850 5200 50  0001 C CNN
+F 4 "https://www.digikey.ca/product-detail/en/adam-tech/PH1-15-UA/2057-PH1-15-UA-ND/9830359" H 3850 5200 50  0001 C CNN "Digikey"
 	1    3850 5200
 	1    0    0    -1
@@
 F 2 "Connector_PinHeader_2.54mm:PinHeader_1x15_P2.54mm_Vertical" H 5000 5250 50  0001 C CNN
 F 3 "~" H 5000 5250 50  0001 C CNN
+F 4 "https://www.digikey.ca/product-detail/en/adam-tech/PH1-15-UA/2057-PH1-15-UA-ND/9830359" H 5000 5250 50  0001 C CNN "Digikey"
 	1    5000 5250
 	1    0    0    -1
@@
 F 3 "~" H 2200 1200 50  0001 C CNN
 F 4 "UWT1H470MCL1GS" H 2200 1200 50  0001 C CNN "Part Number"
+F 5 "https://www.digikey.com/product-detail/en/nichicon/UWT1H470MCL1GS/493-2225-1-ND/590200" H 2200 1200 50  0001 C CNN "Digikey"
 	1    2200 1200
 	-1   0    0    -1
@@
 F 3 "~" H 4100 1200 50  0001 C CNN
 F 4 "UWT1H470MCL1GS" H 4100 1200 50  0001 C CNN "Part Number"
+F 5 "https://www.digikey.com/product-detail/en/nichicon/UWT1H470MCL1GS/493-2225-1-ND/590200" H 4100 1200 50  0001 C CNN "Digikey"
 	1    4100 1200
 	-1   0    0    -1
@@
 F 3 "~" H 5900 1200 50  0001 C CNN
 F 4 "UWT1H470MCL1GS" H 5900 1200 50  0001 C CNN "Part Number"
+F 5 "https://www.digikey.com/product-detail/en/nichicon/UWT1H470MCL1GS/493-2225-1-ND/590200" H 5900 1200 50  0001 C CNN "Digikey"
 	1    5900 1200
 	-1   0    0    -1
